Commit message: all grippers done

File: assets/gripper/rochu_4f/urdf/rochu_4f.urdf (robot description, URDF)
Before this commit: robot finray3f, 4 links, 3 joints
Links:
- added link finger_4_link, mass 0.034805; collision mesh filename=../meshes/finger_4_link.STL; visual mesh filename=../meshes/finger_4_link.STL
- link base_link: mass 0.26864 -> 0.10913
- link finger_1_link: mass 0.039598 -> 0.034805
- link finger_2_link: mass 0.039598 -> 0.034805
- link finger_3_link: mass 0.03 -> 0.034805
Joints:
- added joint finger_4_joint: type revolute, parent base_link, child finger_4_link, origin xyz=0 -0.044 -0.03755 rpy=1.5708 0 1.5708, axis 0 0 1, limit lower=-0.3725 upper=0.785 effort=0.785 velocity=0.785
- joint finger_1_joint: limit lower=0 upper=0.785 effort=0.785 velocity=0.785 -> lower=-0.3725 upper=0.785 effort=0.785 velocity=0.785; origin xyz=0.056 0 -0.014 rpy=1.5708 0.2618 0 -> xyz=0.044 0 -0.03755 rpy=-1.5708 0 0
- joint finger_2_joint: limit lower=0 upper=0.785 effort=0.785 velocity=0.785 -> lower=-0.3725 upper=0.785 effort=0.785 velocity=0.785; origin xyz=-0.028 0.048497 -0.014 rpy=1.5708 0.2618 2.0944 -> xyz=0 0.044 -0.03755 rpy=-1.5708 0 1.5708
- joint finger_3_joint: limit lower=0 upper=0.785 effort=0.785 velocity=0.785 -> lower=-0.3725 upper=0.785 effort=0.785 velocity=0.785; origin xyz=-0.028 -0.048497 -0.014 rpy=-1.5708 -0.2618 1.0472 -> xyz=-0.044 0 -0.03755 rpy=1.5708 0 0
